File: 42Keys/chocorne low_rp2040/chococorne.kicad_pcb (KiCad board)
At the start: 2 copper layers, 130 x 87.7 mm, 63 parts, among them J1 MJ-4PP-9, J2 OLED, SW1 SW_PUSH, SW10 SW_PUSH, SW11 SW_PUSH, SW12 SW_PUSH, SW13 SW_PUSH, SW14 SW_PUSH, SW15 SW_PUSH, SW16 SW_PUSH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

Commit message: add switch and relocate pcb
Parts:
- added ?: , , F.Cu at (185.4, 82.5)
- added REF**: JST_XH_B2B-XH-A_1x02_P2.50mm_Vertical, Connector_JST:JST_XH_B2B-XH-A_1x02_P2.50mm_Vertical, F.Cu at (170.3, 83.2)
- added REF**1: JST_XH_B2B-XH-A_1x02_P2.50mm_Vertical, Connector_JST:JST_XH_B2B-XH-A_1x02_P2.50mm_Vertical, F.Cu at (170.4, 92.7)
- added SW01: SW_SPDT, kicad:switch_SSSS811101, F.Cu at (186.0, 90.0)
- added SW01: SW_SPDT, kicad:switch_SSSS811101, B.Cu at (186.1, 90.1)
- moved RZ1 2.62 mm to (168.3, 76.0)
- moved RZ1 2.61 mm to (187.8, 77.3)
Routing:
- net (no net): track 0.00 -> 60.8 mm, vias 0 -> 2
- net data: track 41.4 -> 76.2 mm
- net GND: track 88.5 -> 102.1 mm
- net VCC: track 91.7 -> 97.6 mm
- net col1: track 175.6 -> 179.4 mm
- net row3: track 87.9 -> 91.6 mm
- net row1: track 153.3 -> 156.8 mm, vias 2 -> 0
- net SDA: track 35.3 -> 38.7 mm
- net col4: track 153.7 -> 157.0 mm, vias 0 -> 2
- net SCL: track 39.0 -> 42.2 mm
- net row2: track 170.7 -> 173.9 mm
- net col3: track 168.4 -> 171.5 mm
- net col2: track 157.0 -> 159.9 mm
- net col5: track 126.8 -> 129.6 mm, vias 1 -> 2
- net row0: track 169.1 -> 171.7 mm
