File: 42Keys/chocorne low_rp2040/chococorne.kicad_sch (KiCad schematic)
At the start: 91 parts, among them J1 MJ-4PP-9, J2 OLED, J6 MJ-4PP-9, J7 OLED, SW1 SW_PUSH, SW10 SW_PUSH, SW11 SW_PUSH, SW12 SW_PUSH, SW13 SW_PUSH, SW14 SW_PUSH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

Commit message: add switch and relocate pcb
Parts:
- removed RZ2: RP2040-Zero, kicad:RP2040-Zero, symbol rp2040-zero:RP2040-Zero
- removed U2: ProMicro, kbd:ProMicro_v2_1side, symbol chococorne-rescue:ProMicro-kbd-corne-light-rescue
- added SW?: SW_SPDT, kicad:switch_SSSS811101, symbol Switch:SW_SPDT
Connections:
- no-connect marks 9 -> 4
